File: alea/alea.kicad_pcb (KiCad board)
At the start: 4 copper layers, 107.1 x 99.9 mm, 48 parts, among them J1 QL_SLOT_DIN41612, J2 Conn_02x17_Odd_Even, J3 Conn_01x03_Pin, Q1 BC548, U0 LM340T-5, U1 68000D, U10 MSM514400D, U11 MSM514400D, U12 DP4873V, U2 EP1810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

Commit message: small update in alea
Connections:
- U8 pad 1: /DG0 -> /DG2
- U8 pad 2: /DG2 -> /DG3
- U8 pad 24: /DG3 -> /DG1
- U8 pad 25: /DG1 -> /DG0
- U9 pad 1: /DG4 -> /DG6
- U9 pad 2: /DG6 -> /DG7
- U9 pad 24: /DG7 -> /DG5
- U9 pad 25: /DG5 -> /DG4
Routing:
- net /DG3: track 129.6 -> 120.3 mm
- net /DG7: track 94.8 -> 86.5 mm
- net /DG4: track 103.5 -> 110.3 mm
- net /DG0: track 130.8 -> 137.2 mm
- net /DTA: track 59.1 -> 53.1 mm
- net /16MHZ: track 52.6 -> 54.4 mm
- net /DG6: track 93.6 -> 92.1 mm
- net /DG2: track 126.3 -> 125.4 mm
- net /DG1: track 131.7 -> 131.0 mm
- net /DG5: track 105.9 -> 105.3 mm
